Commit message: adjusted robot description. fixes #1

File: lwr-robot.urdf (robot description, URDF)
Before this commit: robot lwr, 11 links, 10 joints
Links:
- removed link world_link
Joints:
- removed joint world_lwr_arm_base_joint
- joint arm_world_joint: child world_link -> lwr_arm_base_link; origin xyz=0 0 0.3 rpy=0 0 0 -> xyz=0 0 0.01 rpy=0 0 0

Commit message: better collision model for the arm

File: lwr-robot.urdf (robot description, URDF)
Before this commit: robot lwr, 10 links, 9 joints
Links:
- removed link lwr_tool_mount
- link lwr_arm_7_link: geometry collision mesh filename=package://./meshes/arm_flanche.dae scale=100 100 100; visual mesh filename=package://./meshes/arm_flanche.dae scale=100 100 100
Joints:
- removed joint lwr_arm_hand_fixed_joint

Commit message: urdf: change scaling factors

File: lwr-robot.urdf (robot description, URDF)
Before this commit: robot kuka-lwr, 9 links, 8 joints
Links:
- link lwr_arm_1_link: geometry collision mesh filename=package://./meshes/convex/arm_segment_a_convex.stl scale=1.0 1.0 1.0; visual mesh filename=package://./meshes/arm_segment_a.dae scale=1 1 1
- link lwr_arm_2_link: geometry collision mesh filename=package://./meshes/convex/arm_segment_b_convex.stl scale=1.0 1.0 1.0; visual mesh filename=package://./meshes/arm_segment_b.dae scale=1 1 1
- link lwr_arm_3_link: geometry collision mesh filename=package://./meshes/convex/arm_segment_a_convex.stl scale=1.0 1.0 1.0; visual mesh filename=package://./meshes/arm_segment_a.dae scale=1 1 1
- link lwr_arm_4_link: geometry collision mesh filename=package://./meshes/convex/arm_segment_b_convex.stl scale=1.0 1.0 1.0; visual mesh filename=package://./meshes/arm_segment_b.dae scale=1 1 1
- link lwr_arm_5_link: geometry collision mesh filename=package://./meshes/convex/arm_segment_last_convex.stl scale=1.0 1.0 1.0; visual mesh filename=package://./meshes/arm_segment_last.dae scale=1 1 1
- link lwr_arm_6_link: geometry collision mesh filename=package://./meshes/convex/arm_wrist_convex.stl scale=1.0 1.0 1.0; visual mesh filename=package://./meshes/arm_wrist.dae scale=1 1 1
- link lwr_arm_7_link: geometry collision mesh filename=package://./meshes/arm_flanche.dae scale=1 1 1; visual mesh filename=package://./meshes/arm_flanche.dae scale=1 1 1
- link lwr_arm_base_link: geometry collision mesh filename=package://./meshes/convex/arm_base_convex.stl scale=0.9 0.9 0.9; visual mesh filename=package://./meshes/arm_base.dae scale=1 1 1
